File: 02-module_satellite/02-hardware/home_automation_module_std/home_automation_module_std.kicad_sch (KiCad schematic)
At the start: 25 parts, among them J1 Conn_HE13_1x2_2.54V, J2 Conn_HE13_1x6_2.54H, J3 Conn_HE13_1x6_2.54H, J4 Conn_HE13_1x4_2.54H, J5 Conn_HE13_1x3_2.54V, M1 nRF24L01, Q1 BSS315PH6327XTSA1, Q2 BC848B, U1 TPS70933DBV, U2 TPS70950DBV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

Commit message: [HW] Home automation module PCB v1.0
Parts:
- removed J2, J3: Conn_HE13_1x6_2.54H, p_Package_Misc:PinHeader_1x06_P2.54mm_Horizontal, symbol p_Misc:Conn_HE13_1x6_2.54H
- removed J4: Conn_HE13_1x4_2.54H, p_Package_Misc:PinHeader_1x04_P2.54mm_Horizontal, symbol p_Misc:Conn_HE13_1x4_2.54H
- added J2, J3: Conn_HE13_1x6_2.54V, p_Package_Misc:PinHeader_1x06_P2.54mm_Vertical, symbol p_Misc:Conn_HE13_1x6_2.54V
- added J4: Conn_HE13_1x4_2.54V, p_Package_Misc:PinHeader_1x04_P2.54mm_Vertical, symbol p_Misc:Conn_HE13_1x4_2.54V
Connections:
- net +12V: now also J3.1
- net +3.3V: now also J3.2, J4.1
- net EXT_GPIO: now also J3.5
- net GND: now also J2.2, J2.5, J3.6, J4.4
- net I2C_SCL: now also J3.3
- net I2C_SDA: now also J3.4
- net Input_stage/INPUT1: now also J2.1
- net Input_stage/INPUT2: now also J2.3
- net Input_stage/INPUT3: now also J2.4
- net Input_stage/INPUT4: now also J2.6
- net SWD_CLK: now also J4.3
- net SWD_IO: now also J4.2
- net TEMP_SENSOR_EN renamed LIGHT_SENSOR_EN
Changed lines of the file:
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@@
     (effects (font (size 1.27 1.27)) (justify left bottom))
   )
-  (label "TEMP_SENSOR_EN" (at 267.97 123.19 180) (fields_autoplaced)
+  (label "LIGHT_SENSOR_EN" (at 267.97 123.19 180) (fields_autoplaced)
     (effects (font (size 1.27 1.27)) (justify right bottom))
   )
@@
     (effects (font (size 1.27 1.27)) (justify right bottom))
   )
-  (label "TEMP_SENSOR_EN" (at 205.74 119.38 180) (fields_autoplaced)
+  (label "LIGHT_SENSOR_EN" (at 205.74 119.38 180) (fields_autoplaced)
     (effects (font (size 1.27 1.27)) (justify right bottom))
   )
@@
   (label "SPI_MOSI" (at 215.9 34.29 0) (fields_autoplaced)
     (effects (font (size 1.27 1.27)) (justify left bottom))
-  )
-  (symbol (lib_id "p_Misc:Conn_HE13_1x4_2.54H") (at 24.13 138.43 0) (mirror y) (unit 1)
-    (in_bom yes) (on_board yes) (dnp no)
-    (property "Reference" "J4" (at 20.32 130.81 0)
-      (effects (font (size 1.27 1.27)))
-    )
-    (property "Value" "Conn_HE13_1x4_2.54H" (at 21.59 129.54 0)
-      (effects (font (size 1.27 1.27)) hide)
-    )
-    (property "Footprint" "p_Package_Misc:PinHeader_1x04_P2.54mm_Horizontal" (at 22.86 149.86 0)
-      (effects (font (size 1.27 1.27)) hide)
-    )
-    (property "Datasheet" "" (at 26.67 135.89 0)
-      (effects (font (size 1.27 1.27)) hide)
-    )
-    (pin "1")
-    (pin "2")
-    (pin "3")
-    (pin "4")
-    (instances
-      (project "home_automation_module_std"
-        (path "/b2aa5704-27c4-4dd5-9409-a30bd022abc9"
-          (reference "J4") (unit 1)
-        )
-      )
-    )
   )
   (symbol (lib_id "power:+5V") (at 92.71 41.91 0) (unit 1)
@@
     )
   )
-  (symbol (lib_id "p_Misc:Conn_HE13_1x6_2.54H") (at 26.67 102.87 0) (mirror y) (unit 1)
-    (in_bom yes) (on_board yes) (dnp no)
-    (property "Reference" "J3" (at 20.32 99.06 0)
-      (effects (font (size 1.27 1.27)))
-    )
-    (property "Value" "Conn_HE13_1x6_2.54H" (at 21.59 97.79 0)
-      (effects (font (size 1.27 1.27)) hide)
-    )
-    (property "Footprint" "p_Package_Misc:PinHeader_1x06_P2.54mm_Horizontal" (at 20.32 123.19 0)
-      (effects (font (size 1.27 1.27)) hide)
-    )
-    (property "Datasheet" "" (at 26.67 104.14 0)
-      (effects (font (size 1.27 1.27)) hide)
-    )
-    (pin "1")
-    (pin "2")
-    (pin "3")
-    (pin "4")
-    (pin "5")
-    (pin "6")
-    (instances
-      (project "home_automation_module_std"
-        (path "/b2aa5704-27c4-4dd5-9409-a30bd022abc9"
-          (reference "J3") (unit 1)
-        )
-      )
-    )
-  )
   (symbol (lib_id "p_Passive:R_0603") (at 43.18 161.29 90) (unit 1)
     (in_bom yes) (on_board yes) (dnp no)
@@
         (path "/b327f361-d184-4480-bd5b-3b495e546706"
           (reference "#PWR03") (unit 1)
+        )
+      )
+    )
+  )
+  (symbol (lib_id "p_Misc:Conn_HE13_1x4_2.54V") (at 24.13 138.43 0) (mirror y) (unit 1)
+    (in_bom yes) (on_board yes) (dnp no)
+    (property "Reference" "J4" (at 20.32 130.81 0)
+      (effects (font (size 1.27 1.27)))
+    )
+    (property "Value" "Conn_HE13_1x4_2.54V" (at 17.78 139.7 0)
+      (effects (font (size 1.27 1.27)) (justify left) hide)
+    )
+    (property "Footprint" "p_Package_Misc:PinHeader_1x04_P2.54mm_Vertical" (at 22.86 149.86 0)
+      (effects (font (size 1.27 1.27)) hide)
+    )
+    (property "Datasheet" "" (at 26.67 135.89 0)
+      (effects (font (size 1.27 1.27)) hide)
+    )
+    (pin "1")
+    (pin "2")
+    (pin "3")
+    (pin "4")
+    (instances
+      (project "home_automation_module_std"
+        (path "/b2aa5704-27c4-4dd5-9409-a30bd022abc9"
+          (reference "J4") (unit 1)
         )
       )
@@
     )
   )
-  (symbol (lib_id "p_Misc:Conn_HE13_1x6_2.54H") (at 26.67 69.85 0) (mirror y) (unit 1)
-    (in_bom yes) (on_board yes) (dnp no)
-    (property "Reference" "J2" (at 20.32 66.04 0)
-      (effects (font (size 1.27 1.27)))
-    )
-    (property "Value" "Conn_HE13_1x6_2.54H" (at 21.59 64.77 0)
-      (effects (font (size 1.27 1.27)) hide)
-    )
-    (property "Footprint" "p_Package_Misc:PinHeader_1x06_P2.54mm_Horizontal" (at 20.32 90.17 0)
+  (symbol (lib_id "p_Misc:Conn_HE13_1x3_2.54V") (at 24.13 163.83 0) (mirror y) (unit 1)
+    (in_bom yes) (on_board yes) (dnp no)
+    (property "Reference" "J5" (at 20.32 157.48 0)
+      (effects (font (size 1.27 1.27)))
+    )
+    (property "Value" "Conn_HE13_1x3_2.54V" (at 21.59 156.21 0)
+      (effects (font (size 1.27 1.27)) hide)
+    )
+    (property "Footprint" "p_Package_Misc:PinHeader_1x03_P2.54mm_Vertical" (at 19.05 173.99 0)
+      (effects (font (size 1.27 1.27)) hide)
+    )
+    (property "Datasheet" "" (at 26.67 162.56 0)
+      (effects (font (size 1.27 1.27)) hide)
+    )
+    (pin "1")
+    (pin "2")
+    (pin "3")
+    (instances
+      (project "home_automation_module_std"
+        (path "/b2aa5704-27c4-4dd5-9409-a30bd022abc9"
+          (reference "J5") (unit 1)
+        )
+      )
+    )
+  )
+  (symbol (lib_id "power:+3.3V") (at 92.71 17.78 0) (unit 1)
+    (in_bom yes) (on_board yes) (dnp no)
+    (property "Reference" "#PWR02" (at 92.71 21.59 0)
+      (effects (font (size 1.27 1.27)) hide)
+    )
+    (property "Value" "+3.3V" (at 92.71 13.97 0)
+      (effects (font (size 1.27 1.27)))
+    )
+    (property "Footprint" "" (at 92.71 17.78 0)
+      (effects (font (size 1.27 1.27)) hide)
+    )
+    (property "Datasheet" "" (at 92.71 17.78 0)
+      (effects (font (size 1.27 1.27)) hide)
+    )
+    (pin "1")
+    (instances
+      (project "home_automation_module_std"
+        (path "/b2aa5704-27c4-4dd5-9409-a30bd022abc9"
+          (reference "#PWR02") (unit 1)
+        )
+      )
+    )
+  )
+  (symbol (lib_id "p_Misc:Conn_HE13_1x6_2.54V") (at 26.67 69.85 0) (mirror y) (unit 1)
+    (in_bom yes) (on_board yes) (dnp no)
+    (property "Reference" "J2" (at 21.59 66.04 0)
+      (effects (font (size 1.27 1.27)) (justify left))
+    )
+    (property "Value" "Conn_HE13_1x6_2.54V" (at 17.78 77.47 0)
+      (effects (font (size 1.27 1.27)) (justify left) hide)
+    )
+    (property "Footprint" "p_Package_Misc:PinHeader_1x06_P2.54mm_Vertical" (at 20.32 90.17 0)
       (effects (font (size 1.27 1.27)) hide)
     )
@@
     )
   )
-  (symbol (lib_id "p_Misc:Conn_HE13_1x3_2.54V") (at 24.13 163.83 0) (mirror y) (unit 1)
-    (in_bom yes) (on_board yes) (dnp no)
-    (property "Reference" "J5" (at 20.32 157.48 0)
-      (effects (font (size 1.27 1.27)))
-    )
-    (property "Value" "Conn_HE13_1x3_2.54V" (at 21.59 156.21 0)
-      (effects (font (size 1.27 1.27)) hide)
-    )
-    (property "Footprint" "p_Package_Misc:PinHeader_1x03_P2.54mm_Vertical" (at 19.05 173.99 0)
-      (effects (font (size 1.27 1.27)) hide)
-    )
-    (property "Datasheet" "" (at 26.67 162.56 0)
-      (effects (font (size 1.27 1.27)) hide)
-    )
-    (pin "1")
-    (pin "2")
-    (pin "3")
-    (instances
-      (project "home_automation_module_std"
-        (path "/b2aa5704-27c4-4dd5-9409-a30bd022abc9"
-          (reference "J5") (unit 1)
-        )
-      )
-    )
-  )
-  (symbol (lib_id "power:+3.3V") (at 92.71 17.78 0) (unit 1)
-    (in_bom yes) (on_board yes) (dnp no)
-    (property "Reference" "#PWR02" (at 92.71 21.59 0)
-      (effects (font (size 1.27 1.27)) hide)
-    )
-    (property "Value" "+3.3V" (at 92.71 13.97 0)
-      (effects (font (size 1.27 1.27)))
-    )
-    (property "Footprint" "" (at 92.71 17.78 0)
-      (effects (font (size 1.27 1.27)) hide)
-    )
-    (property "Datasheet" "" (at 92.71 17.78 0)
-      (effects (font (size 1.27 1.27)) hide)
-    )
-    (pin "1")
-    (instances
-      (project "home_automation_module_std"
-        (path "/b2aa5704-27c4-4dd5-9409-a30bd022abc9"
-          (reference "#PWR02") (unit 1)
-        )
-      )
-    )
-  )
   (symbol (lib_id "power:GND") (at 29.21 142.24 90) (unit 1)
     (in_bom yes) (on_board yes) (dnp no)
@@
         )
       )
+    )
+  )
+  (symbol (lib_id "p_Misc:Conn_HE13_1x6_2.54V") (at 26.67 102.87 0) (mirror y) (unit 1)
+    (in_bom yes) (on_board yes) (dnp no)
+    (property "Reference" "J3" (at 20.32 99.06 0)
+      (effects (font (size 1.27 1.27)))
+    )
+    (property "Value" "Conn_HE13_1x6_2.54V" (at 21.59 97.79 0)
+      (effects (font (size 1.27 1.27)) hide)
+    )
+    (property "Footprint" "p_Package_Misc:PinHeader_1x06_P2.54mm_Vertical" (at 20.32 123.19 0)
+      (effects (font (size 1.27 1.27)) hide)
+    )
+    (property "Datasheet" "" (at 26.67 104.14 0)
+      (effects (font (size 1.27 1.27)) hide)
+    )
+    (pin "1")
+    (pin "2")
+    (pin "3")
+    (pin "4")
+    (pin "5")
+    (pin "6")
+    (instances
+      (project "home_automation_module_std"
+        (path "/b2aa5704-27c4-4dd5-9409-a30bd022abc9"
+          (reference "J3") (unit 1)
+        )
+      )
