File: 02-module_satellite/02-hardware/home_automation_module_std/mcu.kicad_sch (KiCad schematic)
At the start: 20 parts, among them J2 Conn_HE13_1x2_2.54V, Q11 2SK1829, U1 STM32G030_C8, Y1 Crystal_3.2x1.5mm

Commit message: [HW] Home automation module PCB v1.0
Parts:
- removed R25: DNP, p_Package_Resistor_SMD:R_0603_1608Metric_Pad0.98x0.95mm_HandSolder, symbol p_Passive:R_0603
Connections:
- net ~{RST}: no longer J2.2, U1.10 (NRST)
- new net ~{NRST}: J2.2, U1.10 (NRST)
Changed lines of the file:
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@@
   (junction (at 128.27 114.3) (diameter 0) (color 0 0 0 0)
   )
-  (junction (at 201.93 39.37) (diameter 0) (color 0 0 0 0)
-  )
   (junction (at 109.22 99.06) (diameter 0) (color 0 0 0 0)
   )
   (junction (at 106.68 43.18) (diameter 0) (color 0 0 0 0)
-  )
-  (junction (at 209.55 39.37) (diameter 0) (color 0 0 0 0)
   )
   (junction (at 80.01 157.48) (diameter 0) (color 0 0 0 0)
@@
     (effects (font (size 1.27 1.27)) (justify right bottom))
   )
-  (label "~{RST}" (at 127 109.22 0) (fields_autoplaced)
+  (label "~{NRST}" (at 127 109.22 0) (fields_autoplaced)
     (effects (font (size 1.27 1.27)) (justify left bottom))
   )
@@
         )
       )
-    )
-  )
-  (symbol (lib_id "p_Passive:R_0603") (at 205.74 39.37 90) (unit 1)
-    (in_bom yes) (on_board yes) (dnp no)
-    (property "Reference" "R25" (at 203.2 36.83 90)
-      (effects (font (size 1.27 1.27)))
-    )
-    (property "Value" "DNP" (at 208.28 36.83 90)
-      (effects (font (size 1.27 1.27)))
-    )
-    (property "Footprint" "p_Package_Resistor_SMD:R_0603_1608Metric_Pad0.98x0.95mm_HandSolder" (at 205.74 39.37 0)
-      (effects (font (size 1.27 1.27)) hide)
-    )
-    (property "Datasheet" "" (at 205.74 39.37 0)
-      (effects (font (size 1.27 1.27)) hide)
-    )
-    (pin "1")
-    (pin "2")
-    (instances
-      (project "home_automation_module_std"
-        (path "/b2aa5704-27c4-4dd5-9409-a30bd022abc9/f6e9616f-65c8-48b9-86d4-91aa35157a80"
-          (reference "R25") (unit 1)
-        )
-      )
