File: 02-module_satellite/02-hardware/four_relays_extension/four_relays_extension.kicad_sch (KiCad schematic)
At the start: 32 parts, among them J1 Conn_HE13_1x3_2.54V, J2 Conn_HE13_1x3_2.54V, J3 Conn_HE13_1x3_2.54V, J4 Conn_HE13_1x3_2.54V, J5 Conn_HE13_1x6_2.54V, K1 Relay SPDT_Type1, K2 Relay SPDT_Type1, K3 Relay SPDT_Type1, K4 Relay SPDT_Type1, Q1 BSS138LT3G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

Commit message: [HW] Home automation four relays extension PCB v1.0
Parts:
- removed H1, H2: drill_hole_5mm, p_Package_Misc:Drill_hole_5mm, symbol p_Misc:drill_hole_5mm
- added H1, H2: drill_hole_2mm_nocu, p_Package_Misc:Drill_hole_2mm_nocu, symbol p_Misc:drill_hole_2mm_nocu
Connections:
- no-connect marks 5 -> 3
Changed lines of the file:
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@@
   (junction (at 92.71 190.5) (diameter 0) (color 0 0 0 0)
   )
-  (no_connect (at 35.56 132.08))
   (no_connect (at 110.49 91.44))
-  (no_connect (at 35.56 135.89))
   (no_connect (at 110.49 96.52))
   (no_connect (at 110.49 93.98))
@@
     )
   )
-  (symbol (lib_id "p_Misc:drill_hole_5mm") (at 33.02 135.89 0) (unit 1)
-    (in_bom yes) (on_board yes) (dnp no)
-    (property "Reference" "H2" (at 27.94 135.89 0)
-      (effects (font (size 1.27 1.27)))
-    )
-    (property "Value" "drill_hole_5mm" (at 31.75 132.08 0)
-      (effects (font (size 1.27 1.27)) hide)
-    )
-    (property "Footprint" "p_Package_Misc:Drill_hole_5mm" (at 33.02 140.97 0)
-      (effects (font (size 1.27 1.27)) hide)
-    )
-    (property "Datasheet" "" (at 33.02 135.89 0)
-      (effects (font (size 1.27 1.27)) hide)
-    )
-    (pin "1")
-    (instances
-      (project "four_relays_extension"
-        (path "/cca46bfc-351e-4628-b687-5558e1401cd2"
-          (reference "H2") (unit 1)
-        )
-      )
-    )
-  )
   (symbol (lib_id "p_Misc:Relay_SPDT_Type1") (at 205.74 82.55 0) (unit 1)
     (in_bom yes) (on_board yes) (dnp no)
@@
         (path "/cca46bfc-351e-4628-b687-5558e1401cd2"
           (reference "J3") (unit 1)
-        )
-      )
-    )
-  )
-  (symbol (lib_id "p_Misc:drill_hole_5mm") (at 33.02 132.08 0) (unit 1)
-    (in_bom yes) (on_board yes) (dnp no)
-    (property "Reference" "H1" (at 27.94 132.08 0)
-      (effects (font (size 1.27 1.27)))
-    )
-    (property "Value" "drill_hole_5mm" (at 31.75 128.27 0)
-      (effects (font (size 1.27 1.27)) hide)
-    )
-    (property "Footprint" "p_Package_Misc:Drill_hole_5mm" (at 33.02 137.16 0)
-      (effects (font (size 1.27 1.27)) hide)
-    )
-    (property "Datasheet" "" (at 33.02 132.08 0)
-      (effects (font (size 1.27 1.27)) hide)
-    )
-    (pin "1")
-    (instances
-      (project "four_relays_extension"
-        (path "/cca46bfc-351e-4628-b687-5558e1401cd2"
-          (reference "H1") (unit 1)
         )
       )
@@
     )
   )
+  (symbol (lib_id "p_Misc:drill_hole_2mm_nocu") (at 33.02 132.08 0) (unit 1)
+    (in_bom yes) (on_board yes) (dnp no)
+    (property "Reference" "H1" (at 27.94 132.08 0)
+      (effects (font (size 1.27 1.27)))
+    )
+    (property "Value" "drill_hole_2mm_nocu" (at 31.75 128.27 0)
+      (effects (font (size 1.27 1.27)) hide)
+    )
+    (property "Footprint" "p_Package_Misc:Drill_hole_2mm_nocu" (at 35.56 134.62 0)
+      (effects (font (size 1.27 1.27)) hide)
+    )
+    (property "Datasheet" "" (at 35.56 132.08 0)
+      (effects (font (size 1.27 1.27)) hide)
+    )
+    (pin "1")
+    (instances
+      (project "four_relays_extension"
+        (path "/cca46bfc-351e-4628-b687-5558e1401cd2"
+          (reference "H1") (unit 1)
+        )
+      )
+    )
+  )
   (symbol (lib_id "p_Passive:C_0603") (at 119.38 76.2 0) (unit 1)
     (in_bom yes) (on_board yes) (dnp no)
@@
         )
       )
+    )
+  )
+  (symbol (lib_id "p_Misc:drill_hole_2mm_nocu") (at 33.02 135.89 0) (unit 1)
+    (in_bom yes) (on_board yes) (dnp no)
+    (property "Reference" "H2" (at 27.94 135.89 0)
+      (effects (font (size 1.27 1.27)))
+    )
+    (property "Value" "drill_hole_2mm_nocu" (at 31.75 132.08 0)
+      (effects (font (size 1.27 1.27)) hide)
+    )
+    (property "Footprint" "p_Package_Misc:Drill_hole_2mm_nocu" (at 35.56 138.43 0)
+      (effects (font (size 1.27 1.27)) hide)
+    )
+    (property "Datasheet" "" (at 35.56 135.89 0)
+      (effects (font (size 1.27 1.27)) hide)
+    )
+    (pin "1")
+    (instances
+      (project "four_relays_extension"
+        (path "/cca46bfc-351e-4628-b687-5558e1401cd2"
+          (reference "H2") (unit 1)
+        )
+      )
